Commit message: moveit collision env/new robot description

File: costar_robot/iiwa14_s_model/urdf/iiwa14_touch_s_model.urdf.xacro (robot description, xacro)
@@ -5,6 +5,7 @@
   <!--Import the lbr iiwa macro -->
   <xacro:include filename="$(find iiwa_description)/urdf/iiwa14.xacro"/>
-  <xacro:include filename="$(find robotiq_s_model_visualization)/cfg/s-model_articulated.urdf"/>
-  <xacro:include filename="$(find robotiq_s_model_visualization)/cfg/s-model_mesh.urdf"/>
+  <!--<xacro:include filename="$(find robotiq_s_model_visualization)/cfg/s-model_mesh.urdf"/>-->
+	<xacro:include filename="$(find robotiq_s_model_visualization)/cfg/s-model_articulated_macro.xacro" />
+	<xacro:s-model_articulated prefix="s_model_"/>
   <!-- Fix to world just for testing -->
   <link name="world"/>
@@ -14,3 +15,8 @@
     <origin xyz="0 0 0.0" rpy="0 0 0" />
   </xacro:iiwa14>
+  <joint name="iiwa_link_ee_to_connector"  type="fixed">
+    <parent link="$(arg robot_name)_link_ee"/>
+    <child link="s_model_palm"/>
+    <origin xyz="0 0 .05" rpy="0.2618 0 0"/>
+  </joint>
 </robot>

Commit message: adding in iiwa14 with s model urdf -- early version

File: costar_robot/iiwa14_s_model/urdf/iiwa14_touch_s_model.urdf.xacro (robot description, xacro)
@@ -1,4 +1,4 @@
 <?xml version="1.0"?>
-<robot name="iiwa14" xmlns:xacro="http://www.ros.org/wiki/xacro">
+<robot name="$(arg robot_name)" xmlns:xacro="http://www.ros.org/wiki/xacro">
   <!-- Import Rviz colors -->
   <xacro:include filename="$(find iiwa_description)/urdf/materials.xacro" />
@@ -6,6 +6,6 @@
   <xacro:include filename="$(find iiwa_description)/urdf/iiwa14.xacro"/>
   <!--<xacro:include filename="$(find robotiq_s_model_visualization)/cfg/s-model_mesh.urdf"/>-->
-	<xacro:include filename="$(find robotiq_s_model_visualization)/cfg/s-model_articulated_macro.xacro" />
-	<xacro:s-model_articulated prefix="s_model_"/>
+  <xacro:include filename="$(find robotiq_s_model_visualization)/cfg/s-model_articulated_macro.xacro" />
+  <xacro:s-model_articulated prefix="$(arg robot_name)_s_model_"/>
   <!-- Fix to world just for testing -->
   <link name="world"/>
@@ -15,8 +15,29 @@
     <origin xyz="0 0 0.0" rpy="0 0 0" />
   </xacro:iiwa14>
-  <joint name="iiwa_link_ee_to_connector"  type="fixed">
-    <parent link="$(arg robot_name)_link_ee"/>
-    <child link="s_model_palm"/>
-    <origin xyz="0 0 .05" rpy="0.2618 0 0"/>
+  <joint name="$(arg robot_name)_link_ee_to_connector"  type="fixed">
+    <parent link="$(arg robot_name)_link_ee_kuka"/>
+    <child link="$(arg robot_name)_s_model_connector"/>
+    <origin xyz="0 0 0.02" rpy="0 0 0"/>
+  </joint>
+  <link name="$(arg robot_name)_s_model_connector">
+    <origin xyz="0 0 0.1" rpy="0 0 0.2618"/>
+    <visual>
+      <geometry>
+        <cylinder length="0.06" radius="0.04"/>
+      </geometry>
+      <material name="blue">
+        <color rgba="0 0 .8 1"/>
+      </material>
+    </visual>
+    <collision>
+      <geometry>
+        <cylinder length="0.06" radius="0.04"/>
+      </geometry>
+    </collision>
+  </link>
+  <joint name="$(arg robot_name)_connector_to_palm"  type="fixed">
+    <parent link="$(arg robot_name)_s_model_connector"/>
+    <child link="$(arg robot_name)_s_model_palm"/>
+    <origin xyz="0 0 0.08" rpy="1.5707 0 0"/>
   </joint>
 </robot>

Commit message: robot model with dumb mesh instead of articulated

File: costar_robot/iiwa14_s_model/urdf/iiwa14_touch_s_model.urdf.xacro (robot description, xacro)
@@ -6,6 +6,7 @@
   <xacro:include filename="$(find iiwa_description)/urdf/iiwa14.xacro"/>
   <!--<xacro:include filename="$(find robotiq_s_model_visualization)/cfg/s-model_mesh.urdf"/>-->
-  <xacro:include filename="$(find robotiq_s_model_visualization)/cfg/s-model_articulated_macro.xacro" />
-  <xacro:s-model_articulated prefix="$(arg robot_name)_s_model_"/>
+  <!--<xacro:include filename="$(find robotiq_s_model_visualization)/cfg/s-model_articulated_macro.xacro" />-->
+  <xacro:include filename="$(find robotiq_s_model_visualization)/cfg/s-model_mesh_macro.xacro" />
+  <xacro:s-model_mesh prefix="$(arg robot_name)_s_model_"/>
   <!-- Fix to world just for testing -->
   <link name="world"/>
@@ -36,8 +37,17 @@
     </collision>
   </link>
-  <joint name="$(arg robot_name)_connector_to_palm"  type="fixed">
-    <parent link="$(arg robot_name)_s_model_connector"/>
-    <child link="$(arg robot_name)_s_model_palm"/>
-    <origin xyz="0 0 0.08" rpy="1.5707 0 0"/>
-  </joint>
+  <xacro:if value="false">
+    <joint name="$(arg robot_name)_connector_to_palm"  type="fixed">
+      <parent link="$(arg robot_name)_s_model_connector"/>
+      <child link="$(arg robot_name)_s_model_palm"/>
+      <origin xyz="0 0 0.08" rpy="1.5707 0 0"/>
+    </joint>
+  </xacro:if>
+  <xacro:unless value="false">
+    <joint name="$(arg robot_name)_connector_to_palm"  type="fixed">
+      <parent link="$(arg robot_name)_s_model_connector"/>
+      <child link="$(arg robot_name)_s_model_palm"/>
+      <origin xyz="0 0 0.18" rpy="0 0 3.14159"/>
+    </joint>
+  </xacro:unless>
 </robot>

Commit message: adding 15 degree rotation

File: costar_robot/iiwa14_s_model/urdf/iiwa14_touch_s_model.urdf.xacro (robot description, xacro)
@@ -48,5 +48,5 @@
       <parent link="$(arg robot_name)_s_model_connector"/>
       <child link="$(arg robot_name)_s_model_palm"/>
-      <origin xyz="0 0 0.18" rpy="0 0 3.14159"/>
+      <origin xyz="0 0 0.18" rpy="0 0 ${3.14159+0.2618}"/>
     </joint>
   </xacro:unless>
